File: working/Tiny-Pogo-AVR/Tiny-Pogo-AVR.sch (KiCad schematic (older format))
At the start: 0 parts

Commit message: Release 1
A first release of the designs for the 2.54mm version of the board, with all the design files needed for manufacture.
Parts:
- added C1, C3, C4: 1u, Capacitor_SMD:C_0603_1608Metric, symbol KEMET_SMD:1u_0603
- added C2, C5, C6, C7, C8: 100n, Capacitor_SMD:C_0603_1608Metric, symbol KEMET_SMD:100n_0603
- added D1, D2: LED_Red, LED_SMD:LED_0603_1608Metric, symbol Kingbright:LED_Red_0603
- added D3, D4, D5, D6: LED_Green, LED_SMD:LED_0603_1608Metric, symbol Kingbright:LED_Green_0603
- added H1, H2: MH_M3, MountingHole:MountingHole_3.2mm_M3_Pad_Via, symbol Mechanical:MountingHole_Pad
- added J1: Conn_02x03_Odd_Even, HRG-KICAD-FOOTP-LIB:PogoPin 2x6, symbol Connector_Generic:Conn_02x03_Odd_Even
- added J2: USB_B_Mini, HRG-KICAD-FOOTP-LIB:USB_Mini-B_Wuerth_65100516121_Horizontal, symbol Connector:USB_B_Mini
- added J3: Conn_02x03_Odd_Even, Connector_PinHeader_2.54mm:PinHeader_2x03_P2.54mm_Vertical, symbol Connector_Generic:Conn_02x03_Odd_Even
- added JP1: SolderJumper_2_Open, Jumper:SolderJumper-2_P1.3mm_Open_Pad1.0x1.5mm, symbol Jumper:SolderJumper_2_Open
- added R1: 0R, Resistor_SMD:R_0603_1608Metric, symbol Vishay_Res_SMD:0R_0603
- added R2, R3: 10K, Resistor_SMD:R_0603_1608Metric, symbol Vishay_Res_SMD:10K_0603
- added R4, R5, R6, R7, R8, R9: 330R, Resistor_SMD:R_0603_1608Metric, symbol Vishay_Res_SMD:330R_0603
- added SW1, SW2: SW_SPDT, HRG-KICAD-FOOTP-LIB:CAS-120-B-type, symbol Switch:SW_SPDT
- added U1: ATtiny44A-SSU, Package_SO:SOIC-14_3.9x8.7mm_P1.27mm, symbol MCU_Microchip_ATtiny:ATtiny44A-SSU
- added U2: MIC5317-3.3YM5-TR, HRG-KICAD-FOOTP-LIB:SOT-23-5, symbol HRG-KICAD-SCHEM-LIB:MIC5317-3.3YM5-TR
- added U3, U4: TXB0101DCKR, HRG-KICAD-FOOTP-LIB:SC70-6, symbol HRG-KICAD-SCHEM-LIB:TXB0101DCKR
- added Y1: 20MHz, Crystal:Resonator_muRata_DSS6-3Pin_W7.0mm_H2.5mm, symbol Device:Resonator
Connections:
- new net: JP1.1 (A), R1.2, U1.4 (~RESET~/PB3)
- new net: J2.3 (D+), U3.4 (B)
- new net: R2.2, U3.5 (OE)
- new net: J2.2 (D-), U4.4 (B)
- new net: R3.2, U4.5 (OE)
- new net: D1.1 (K), R4.1
- new net: D2.1 (K), R5.1
- new net: D3.1 (K), R6.2
- new net: D4.1 (K), R7.2
- new net: D5.1 (K), R8.2
- new net: D6.1 (K), R9.2
- new net +3V3: C4.1, C7.1, C8.1, SW2.1 (A), U2.5 (VOUT), U3.6 (VCCB), U4.6 (VCCB)
- new net D+: U1.5 (PB2), U1.6 (PA7), U3.3 (A)
- new net D-: U1.13 (AREF/PA0), U4.3 (A)
- new net GND: C1.2, C2.2, C3.2, C4.2, C5.2, C6.2, C7.2, C8.2, H1.1, H2.1, J1.5 (Pin_5), J2.5 (GND), J3.5 (Pin_5), R4.2, R5.2, R6.1, R7.1, R8.1, R9.1, U1.14 (GND), U2.2 (GND), U3.2 (GND), U4.2 (GND), Y1.2
- new net MISO: D3.2 (A), J1.2 (Pin_2), J3.2 (Pin_2), U1.8 (PA5)
- new net MOSI: D4.2 (A), J1.3 (Pin_3), J3.3 (Pin_3), U1.7 (PA6)
- new net RST: D6.2 (A), J1.6 (Pin_6), J3.6 (Pin_6), JP1.2 (B), U1.10 (PA3)
- new net SCK: D5.2 (A), J1.4 (Pin_4), J3.4 (Pin_4), U1.9 (PA4)
- new net TARGET_VCC: D2.2 (A), J1.1 (Pin_1), J3.1 (Pin_1), SW1.2 (B)
- new net VBUS: C3.1, C5.1, C6.1, D1.2 (A), J2.1 (VBUS), R2.1, R3.1, SW2.3 (C), U2.1 (VIN), U2.3 (EN)
- new net VCC: C1.1, C2.1, R1.1, SW1.1 (A), SW2.2 (B), U1.1 (VCC), U3.1 (VCCA), U4.1 (VCCA)
- new net XTAL1: U1.2 (XTAL1/PB0), Y1.1
- new net XTAL2: U1.3 (XTAL2/PB1), Y1.3
- no-connect marks 0 -> 5
